Commit message: Fix objects spawning

File: adversarial_coverage/objects/obstacle.urdf.xacro (robot description, xacro)
@@ -7,10 +7,10 @@
   <link name="obstacle" type="fixed">
     <inertial>
-      <origin xyz="$(arg row) $(arg col) 0" />
+      <origin xyz="$(arg row) $(arg col) 0.5" />
       <mass value="1.0" />
       <inertia  ixx="0.0" ixy="0.0"  ixz="0.0"  iyy="0.0"  iyz="0.0"  izz="0.0" />
     </inertial>
     <visual>
-      <origin xyz="$(arg row) $(arg col) 0"/>
+      <origin xyz="$(arg row) $(arg col) 0.5"/>
       <geometry>
         <box size="$(arg width) $(arg height) 1" />
@@ -18,5 +18,5 @@
     </visual>
     <collision>
-      <origin xyz="$(arg row) $(arg col) 0"/>
+      <origin xyz="$(arg row) $(arg col) 0.5"/>
       <geometry>
         <box size="$(arg width) $(arg height) 1" />
@@ -24,5 +24,5 @@
     </collision>
   </link>
-  <gazebo reference="obstacle">
+  <gazebo>
     <static>true</static>
     <material>Gazebo/Black</material>
